Commit message: Add files via upload

File: mp_400.urdf (robot description, URDF)
Before this commit: robot mp_400, 32 links, 31 joints
Links:
- removed link arm_0_link
- removed link arm_mount
- removed link laserscanner_back_link
- removed link laserscanner_front_link
- removed link schunk_base_link
- added link arm_base_link, mass 0.01
- added link arm_podest_link, mass 0.01; collision mesh filename=package://schunk_description/meshes/lwa4p/arm_base_link.stl; visual mesh filename=package://schunk_description/meshes/lwa4p/arm_base_link.stl
- added link my_box, mass 0.1; collision box size=0.37 0.05 0.3; visual box size=0.05 0.05 0.3
- added link my_box_1, mass 0.1; collision box size=0.05 0.05 0.3; visual box size=0.05 0.05 0.3
- added link pg70_finger_right_link; collision box size=0.03 0.01 0.01; visual box size=0.03 0.01 0.01
- added link pg70_fingertip_right_link; collision box size=0.03 0.01 0.1; visual box size=0.03 0.01 0.1
- link arm_1_link: mass 0.29364 -> 0.01; geometry collision mesh filename=package://schunk_description/meshes/lwa4p/arm_1_link.stl; visual mesh filename=package://schunk_description/meshes/lwa4p/arm_1_link.stl
- link arm_2_link: mass 0.29364 -> 0.01; geometry collision mesh filename=package://schunk_description/meshes/lwa4p/arm_2_link.stl; visual mesh filename=package://schunk_description/meshes/lwa4p/arm_2_link.stl
- link arm_3_link: mass 0.29364 -> 0.01; geometry collision mesh filename=package://schunk_description/meshes/lwa4p/arm_3_link.stl; visual mesh filename=package://schunk_description/meshes/lwa4p/arm_3_link.stl
- link arm_4_link: mass 0.19364 -> 0.01; geometry collision mesh filename=package://schunk_description/meshes/lwa4p/arm_4_link.stl; visual mesh filename=package://schunk_description/meshes/lwa4p/arm_4_link.stl
- link arm_5_link: mass 0.15364 -> 0.01; geometry collision mesh filename=package://schunk_description/meshes/lwa4p/arm_5_link.stl; visual mesh filename=package://schunk_description/meshes/lwa4p/arm_5_link.stl
- link arm_6_link: mass 0.10364 -> 0.01; geometry collision mesh filename=package://schunk_description/meshes/lwa4p/arm_6_link.stl; visual mesh filename=package://schunk_description/meshes/lwa4p/arm_6_link.stl
- link base_link: mass 30 -> None
- link pg70_finger_left_link: mass 0.1 -> None
- link pg70_fingertip_left_link: mass 0.1 -> None
- link pg70_palm_link: mass 0.1 -> None
Joints:
- removed joint arm_0_joint
- removed joint arm_robot_joint
- removed joint baselink_to_arm_mount
- removed joint laserscanner_back_joint
- removed joint laserscanner_front_joint
- added joint My_box_bottom_joint: type fixed, parent base_link, child my_box, origin xyz=0.23 0 0.315 rpy=0 0 0
- added joint My_box_bottom_joint_1: type fixed, parent base_link, child my_box_1, origin xyz=0.37 0 0.340 rpy=0 0 0
- added joint arm_base_joint: type fixed, parent arm_podest_link, child arm_base_link, origin xyz=0 0 0.10 rpy=0 0 0
- added joint arm_podest_joint: type fixed, parent base_link, child arm_podest_link, origin xyz=0 0 0.7 rpy=0 0 0
- added joint pg70_finger_right_joint: type prismatic, parent pg70_palm_link, child pg70_finger_right_link, origin xyz=0 0 0.0789 rpy=-0 0 0, axis 0 -1 0, limit lower=-0.001 upper=0.04 effort=100 velocity=2.0, mimic joint=pg70_finger_left_joint multiplier=1 offset=0
- added joint pg70_fingertip_right_joint: type fixed, parent pg70_finger_right_link, child pg70_fingertip_right_link, origin xyz=0 -0.01 0.045 rpy=0 0 0
- joint arm_1_joint: limit lower=-2.95 upper=2.95 effort=300 velocity=1.25 -> lower=-2.94 upper=2.94 effort=370 velocity=2.0; origin xyz=0 0 0.11 rpy=0 0 0 -> xyz=0 0 0 rpy=0 0 0; parent arm_0_link -> arm_base_link
- joint arm_2_joint: limit lower=-2.95 upper=2.95 effort=250 velocity=1.25 -> lower=-2.94 upper=2.94 effort=370 velocity=2.0
- joint arm_3_joint: limit lower=-2.95 upper=2.95 effort=200 velocity=1.25 -> lower=-2.68 upper=2.68 effort=176 velocity=2.0
- joint arm_4_joint: limit lower=-2.95 upper=2.95 effort=150 velocity=1.25 -> lower=-2.94 upper=2.94 effort=176 velocity=2.0
- joint arm_5_joint: limit lower=-2.95 upper=2.95 effort=100 velocity=1.25 -> lower=-2.94 upper=2.94 effort=41.6 velocity=2.0
- joint arm_6_joint: limit lower=-2.947 upper=2.947 effort=50 velocity=1.25 -> lower=-2.94 upper=2.94 effort=20.1 velocity=2.0
- joint camera_joint: origin xyz=0.2 0 0 rpy=0 0 0 -> xyz=-0.22 0 0.365 rpy=0 0 0; parent schunk_base_link -> my_box_1
