Commit message: Add files via upload

File: robot.urdf (robot description, URDF)
Before this commit: robot lwa4p, 9 links, 8 joints
Links:
- removed link arm_1_link
- removed link arm_2_link
- removed link arm_3_link
- removed link arm_4_link
- removed link arm_5_link
- removed link arm_6_link
- removed link arm_base_link
- removed link arm_podest_link
- added link pg70_finger_left_link, mass 1; collision box size=0.03 0.01 0.01; visual box size=0.03 0.01 0.01
- added link pg70_finger_right_link, mass 1; collision box size=0.03 0.01 0.01; visual box size=0.03 0.01 0.01
- added link pg70_palm_link, mass 1; collision box size=0.082 0.114 0.080; visual mesh filename=package://schunk_description/meshes/pg70/pg70.dae
- added link pg70_podest_link, mass 0.01; collision mesh filename=package://schunk_description/meshes/lwa4p/arm_base_link.stl; visual mesh filename=package://schunk_description/meshes/lwa4p/arm_base_link.stl
Joints:
- removed joint arm_1_joint
- removed joint arm_2_joint
- removed joint arm_3_joint
- removed joint arm_4_joint
- removed joint arm_5_joint
- removed joint arm_6_joint
- removed joint arm_base_joint
- removed joint arm_podest_joint
- added joint pg70_finger_left_joint: type prismatic, parent pg70_palm_link, child pg70_finger_left_link, origin xyz=0 0 0.0789 rpy=0 0 0, axis 0 1 0, limit lower=-0.001 upper=0.0301 effort=10 velocity=0.041
- added joint pg70_finger_right_joint: type prismatic, parent pg70_palm_link, child pg70_finger_right_link, origin xyz=0 0 0.0789 rpy=-0 0 0, axis 0 -1 0, limit lower=-0.001 upper=0.0301 effort=10 velocity=0.041, mimic joint=pg70_finger_left_joint multiplier=1 offset=0
- added joint pg70_palm_joint: type fixed, parent pg70_podest_link, child pg70_palm_link, origin xyz=0 0 0.10 rpy=0 0 0
- added joint pg70_podest_joint: type fixed, parent world, child pg70_podest_link, origin xyz=0 0 0.026 rpy=0 0 0

Commit message: Update robot.urdf

File: robot.urdf (robot description, URDF)
Before this commit: robot lwa4p, 14 links, 13 joints
Joints:
- joint pg70_finger_right_joint: mimic (none) -> joint=${pg70_finger_left_joint multiplier=1 offset=0

Commit message: Update robot.urdf

File: robot.urdf (robot description, URDF)
Before this commit: robot lwa4p, 14 links, 13 joints
Joints:
- joint pg70_finger_right_joint: mimic joint=${pg70_finger_left_joint multiplier=1 offset=0 -> joint=pg70_finger_left_joint multiplier=1 offset=0

Commit message: Update robot.urdf

File: robot.urdf (robot description, URDF)
Before this commit: robot lwa4p, 14 links, 13 joints
Links:
- removed link world
- added link base_link; collision mesh filename=package://neo_mp_400/robot_model/mp_400/meshes/MP-400-BODY.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 scale=0.001 0.001 0.001; visual mesh filename=package://neo_mp_400/robot_model/mp_400/meshes/MP-400-BODY.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 scale=0.001 0.001 0.001
- added link camera_color_frame
- added link camera_color_optical_frame
- added link camera_depth_frame
- added link camera_depth_optical_frame
- added link camera_left_ir_frame
- added link camera_left_ir_optical_frame
- added link camera_link, mass 0.564; collision box size=0.02505 0.09 0.025; visual mesh filename=package://mp400_description/meshes/d435_camera/d435.dae
- added link camera_right_ir_frame
- added link camera_right_ir_optical_frame
- added link fixed_wheel_left_link, mass 5.3; collision mesh filename=package://neo_mp_400/robot_model/mp_400/meshes/MP-400-FIXED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 scale=0.001 0.001 0.001; visual mesh filename=package://neo_mp_400/robot_model/mp_400/meshes/MP-400-FIXED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 scale=0.001 0.001 0.001
- added link fixed_wheel_right_link, mass 5.3; collision mesh filename=package://neo_mp_400/robot_model/mp_400/meshes/MP-400-FIXED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 scale=0.001 0.001 0.001; visual mesh filename=package://neo_mp_400/robot_model/mp_400/meshes/MP-400-FIXED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 scale=0.001 0.001 0.001
- added link imu_1_link, mass 0.001
- added link lidar_1_link, mass 0.001; collision mesh filename=package://neo_mp_400/robot_model/mp_400/meshes/SICK-S300.dae scale=0.001 0.001 0.001; visual mesh filename=package://neo_mp_400/robot_model/mp_400/meshes/SICK-S300.dae scale=0.001 0.001 0.001
- added link my_box, mass 0.1; collision box size=0.37 0.05 0.3; visual box size=0.05 0.05 0.3
- added link my_box_1, mass 0.1; collision box size=0.05 0.05 0.3; visual box size=0.05 0.05 0.3
- added link wheel_back_left_link, mass 3.5; collision mesh filename=package://neo_mp_400/robot_model/mp_400/meshes/MP-400-CASTE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 scale=0.001 0.001 0.001; visual mesh filename=package://neo_mp_400/robot_model/mp_400/meshes/MP-400-CASTE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 scale=0.001 0.001 0.001
- added link wheel_back_right_link, mass 3.5; collision mesh filename=package://neo_mp_400/robot_model/mp_400/meshes/MP-400-CASTE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 scale=0.001 0.001 0.001; visual mesh filename=package://neo_mp_400/robot_model/mp_400/meshes/MP-400-CASTE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 scale=0.001 0.001 0.001
- added link wheel_front_left_link, mass 3.5; collision mesh filename=package://neo_mp_400/robot_model/mp_400/meshes/MP-400-CASTE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 scale=0.001 0.001 0.001; visual mesh filename=package://neo_mp_400/robot_model/mp_400/meshes/MP-400-CASTE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 scale=0.001 0.001 0.001
- added link wheel_front_right_link, mass 3.5; collision mesh filename=package://neo_mp_400/robot_model/mp_400/meshes/MP-400-CASTE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 scale=0.001 0.001 0.001; visual mesh filename=package://neo_mp_400/robot_model/mp_400/meshes/MP-400-CASTE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 scale=0.001 0.001 0.001
Joints:
- added joint My_box_bottom_joint: type fixed, parent base_link, child my_box, origin xyz=0.23 0 0.315 rpy=0 0 0
- added joint My_box_bottom_joint_1: type fixed, parent base_link, child my_box_1, origin xyz=0.37 0 0.340 rpy=0 0 0
- added joint camera_color_joint: type fixed, parent camera_depth_frame, child camera_color_frame, origin xyz=0 0.015 0 rpy=0 0 0
- added joint camera_color_optical_joint: type fixed, parent camera_color_frame, child camera_color_optical_frame, origin xyz=0 0 0 rpy=-1.57079632679 0 -1.57079632679
- added joint camera_depth_joint: type fixed, parent camera_link, child camera_depth_frame, origin xyz=0.0149 0.0175 0.0125 rpy=0 0 0
- added joint camera_depth_optical_joint: type fixed, parent camera_depth_frame, child camera_depth_optical_frame, origin xyz=0 0 0 rpy=-1.57079632679 0 -1.57079632679
- added joint camera_joint: type fixed, parent base_link, child camera_link, origin xyz=0.15 0 0.705 rpy=0 -0.7 0
- added joint camera_left_ir_joint: type fixed, parent camera_depth_frame, child camera_left_ir_frame, origin xyz=0 0.0 0 rpy=0 0 0
- added joint camera_left_ir_optical_joint: type fixed, parent camera_left_ir_frame, child camera_left_ir_optical_frame, origin xyz=0 0 0 rpy=-1.57079632679 0 -1.57079632679
- added joint camera_right_ir_joint: type fixed, parent camera_depth_frame, child camera_right_ir_frame, origin xyz=0 -0.05 0 rpy=0 0 0
- added joint camera_right_ir_optical_joint: type fixed, parent camera_right_ir_frame, child camera_right_ir_optical_frame, origin xyz=0 0 0 rpy=-1.57079632679 0 -1.57079632679
- added joint fixed_wheel_left_joint: type fixed, parent base_link, child fixed_wheel_left_link, origin xyz=-0. 0.26 0.075 rpy=0 0 1.57, axis 0 1 0, limit lower=-1e+16 upper=1e+16 effort=1000.0 velocity=3.5
- added joint fixed_wheel_right_joint: type fixed, parent base_link, child fixed_wheel_right_link, origin xyz=0. -0.26 0.075 rpy=0 0 -1.57, axis 0 1 0, limit lower=-1e+16 upper=1e+16 effort=1000.0 velocity=3.5
- added joint imu_1_joint: type fixed, parent base_link, child imu_1_link, origin xyz=0.100 0 0.300 rpy=0 0 3.14, axis 0 1 0
- added joint lidar_1_joint: type fixed, parent base_link, child lidar_1_link, origin xyz=0.230 0 0.110 rpy=0 3.14 3.14, axis 0 1 0
- added joint wheel_back_left_joint: type fixed, parent base_link, child wheel_back_left_link, origin xyz=-0.220 0.155 0.036 rpy=0 0 1.57, axis 0 1 0, limit lower=-1e+16 upper=1e+16 effort=1000.0 velocity=3.5
- added joint wheel_back_right_joint: type fixed, parent base_link, child wheel_back_right_link, origin xyz=-0.220 -0.155 0.036 rpy=0 0 1.57, axis 0 1 0, limit lower=-1e+16 upper=1e+16 effort=1000.0 velocity=3.5
- added joint wheel_front_left_joint: type fixed, parent base_link, child wheel_front_left_link, origin xyz=0.165 0.155 0.036 rpy=0 0 1.57, axis 0 1 0, limit lower=-1e+16 upper=1e+16 effort=1000.0 velocity=3.5
- added joint wheel_front_right_joint: type fixed, parent base_link, child wheel_front_right_link, origin xyz=0.165 -0.155 0.036 rpy=0 0 1.57, axis 0 1 0, limit lower=-1e+16 upper=1e+16 effort=1000.0 velocity=3.5
- joint arm_podest_joint: origin xyz=0 0 0.052 rpy=0 0 0 -> xyz=0 0 0.7 rpy=0 0 0; parent world -> base_link
